Commit message: modify the urdf and srdf to fit the walking pattern generator needs

File: simple_humanoid_description/urdf/simple_humanoid.urdf (robot description, URDF)
Before this commit: robot simple_humanoid, 31 links, 30 joints
Links:
- removed link LARM_LINK7
- removed link LLEG_LINK6
- removed link RARM_LINK7
- removed link RLEG_LINK6
- removed link WAIST_LINK0
- removed link WAIST_LINK3
- added link BODY, mass 27
- added link l_ankle, mass 1.9
- added link l_wrist, mass 0.4
- added link r_ankle, mass 1.9
- added link r_wrist, mass 0.4
- added link torso, mass 13
Joints:
- joint CHEST: child WAIST_LINK3 -> torso
- joint LARM_SHOULDER_P: parent WAIST_LINK3 -> torso
- joint LARM_WRIST_R: child LARM_LINK7 -> l_wrist
- joint LLEG_ANKLE_R: child LLEG_LINK6 -> l_ankle
- joint LLEG_HIP_R: parent WAIST_LINK0 -> BODY
- joint RARM_SHOULDER_P: parent WAIST_LINK3 -> torso
- joint RARM_WRIST_R: child RARM_LINK7 -> r_wrist
- joint RLEG_ANKLE_R: child RLEG_LINK6 -> r_ankle
- joint RLEG_HIP_R: parent WAIST_LINK0 -> BODY
- joint WAIST_P: parent WAIST_LINK0 -> BODY
- joint waist: child WAIST_LINK0 -> BODY
