Commit message: Fix wrong limits on simple_humanoid.urdf. Propose a new humanoid model with a standard structure. (simple_humanoid_classical)

File: urdf/simple_humanoid_classical.urdf (robot description, URDF)
Before this commit: robot simple_humanoid, 31 links, 30 joints
Joints:
- joint LLEG_HIP_P: child LLEG_LINK2 -> LLEG_LINK3; limit lower=-0.349065850399 upper=1.57079632679 effort=100 velocity=3.87 -> lower=-0.5236 upper=0.5236 effort=160 velocity=5.8; parent LLEG_LINK1 -> LLEG_LINK2
- joint LLEG_HIP_R: child LLEG_LINK1 -> LLEG_LINK2; origin xyz=0 0.09 0 rpy=0 0 0 -> xyz=0 0 0 rpy=0 0 0; parent BODY -> LLEG_LINK1
- joint LLEG_HIP_Y: child LLEG_LINK3 -> LLEG_LINK1; limit lower=-0.5236 upper=0.5236 effort=160 velocity=5.8 -> lower=-0.349065850399 upper=1.57079632679 effort=100 velocity=3.87; origin xyz=0 0 -0.3535 rpy=0 0 0 -> xyz=0 0.09 0 rpy=0 0 0; parent LLEG_LINK2 -> BODY
- joint LLEG_KNEE: origin xyz=0 0 0 rpy=0 0 0 -> xyz=0 0 -0.3535 rpy=0 0 0
- joint RLEG_HIP_P: child RLEG_LINK2 -> RLEG_LINK3; limit lower=-0.5236 upper=0.5236 effort=160 velocity=5.8 -> lower=-2.095 upper=0.7 effort=160 velocity=5.8; parent RLEG_LINK1 -> RLEG_LINK2
- joint RLEG_HIP_R: child RLEG_LINK1 -> RLEG_LINK2; limit lower=-0.349065850399 upper=1.57079632679 effort=100 velocity=3.87 -> lower=-0.5236 upper=0.5236 effort=160 velocity=5.8; origin xyz=0 -0.09 0 rpy=0 0 0 -> xyz=0 0 0 rpy=0 0 0; parent BODY -> RLEG_LINK1
- joint RLEG_HIP_Y: child RLEG_LINK3 -> RLEG_LINK1; limit lower=-2.095 upper=0.7 effort=160 velocity=5.8 -> lower=-0.349065850399 upper=1.57079632679 effort=100 velocity=3.87; origin xyz=0 0 -0.3535 rpy=0 0 0 -> xyz=0 -0.09 0 rpy=0 0 0; parent RLEG_LINK2 -> BODY
- joint RLEG_KNEE: origin xyz=0 0 0 rpy=0 0 0 -> xyz=0 0 -0.3535 rpy=0 0 0
