Commit message: [urdf] Add limits for each joint.

File: urdf/simple_humanoid.urdf (robot description, URDF)
Before this commit: robot simple_humanoid, 31 links, 30 joints
Joints:
- joint LARM_ELBOW: limit lower=0 upper=0 effort=30 velocity=0 -> lower=-2.42600766027 upper=2.42600766027 effort=70.0 velocity=4.58
- joint LARM_SHOULDER_P: limit lower=0 upper=0 effort=30 velocity=0 -> lower=-1.57079632679 upper=0.785398163397 effort=100.0 velocity=2.7
- joint LARM_SHOULDER_R: limit lower=0 upper=0 effort=30 velocity=0 -> lower=0.00872664625997 upper=2.87106661953 effort=100.0 velocity=3.66
- joint LARM_SHOULDER_Y: limit lower=0 upper=0 effort=30 velocity=0 -> lower=-1.57079632679 upper=0.785398163397 effort=100.0 velocity=2.7
- joint LARM_WRIST_P: limit lower=0 upper=0 effort=30 velocity=0 -> lower=-2.51327412287 upper=2.51327412287 effort=20.0 velocity=1.95
- joint LARM_WRIST_R: limit lower=0 upper=0 effort=30 velocity=0 -> lower=-1.37008346282 upper=1.37008346282 effort=8.0 velocity=1.76
- joint LARM_WRIST_Y: limit lower=0 upper=0 effort=30 velocity=0 -> lower=-2.23402144255 upper=0.00349065850399 effort=70.0 velocity=4.58
- joint LLEG_ANKLE_P: limit lower=0 upper=0 effort=30 velocity=0 -> lower=0 upper=2.618 effort=300 velocity=7
- joint LLEG_ANKLE_R: limit lower=0 upper=0 effort=30 velocity=0 -> lower=-1.27 upper=0.68 effort=160 velocity=5.8
- joint LLEG_HIP_P: limit lower=0 upper=0 effort=30 velocity=0 -> lower=-0.349065850399 upper=1.57079632679 effort=100 velocity=3.87
- joint LLEG_HIP_R: limit lower=0 upper=0 effort=30 velocity=0 -> lower=-0.349065850399 upper=1.57079632679 effort=100 velocity=3.87
- joint LLEG_HIP_Y: limit lower=0 upper=0 effort=30 velocity=0 -> lower=-0.5236 upper=0.5236 effort=160 velocity=5.8
- joint LLEG_KNEE: limit lower=0 upper=0 effort=30 velocity=0 -> lower=-2.095 upper=0.7 effort=160 velocity=5.8
- joint RARM_ELBOW: limit lower=0 upper=0 effort=30 velocity=0 -> lower=-2.23402144255 upper=0.00349065850399 effort=70.0 velocity=4.58
- joint RARM_SHOULDER_P: limit lower=0 upper=0 effort=30 velocity=0 -> lower=-1.57079632679 upper=0.785398163397 effort=100.0 velocity=2.7
- joint RARM_SHOULDER_R: limit lower=0 upper=0 effort=30 velocity=0 -> lower=0.00872664625997 upper=2.87106661953 effort=100.0 velocity=3.66
- joint RARM_SHOULDER_Y: limit lower=0 upper=0 effort=30 velocity=0 -> lower=-2.42600766027 upper=2.42600766027 effort=70.0 velocity=4.58
- joint RARM_WRIST_P: limit lower=0 upper=0 effort=30 velocity=0 -> lower=-1.37008346282 upper=1.37008346282 effort=8.0 velocity=1.76
- joint RARM_WRIST_R: limit lower=0 upper=0 effort=30 velocity=0 -> lower=-0.680678408278 upper=0.680678408278 effort=8.0 velocity=1.76
- joint RARM_WRIST_Y: limit lower=0 upper=0 effort=30 velocity=0 -> lower=-2.51327412287 upper=2.51327412287 effort=20.0 velocity=1.95
- joint RLEG_ANKLE_R: limit lower=0 upper=0 effort=30 velocity=0 -> lower=-1.27 upper=0.68 effort=160 velocity=5.8
- joint RLEG_HIP_P: limit lower=0 upper=0 effort=30 velocity=0 -> lower=-0.5236 upper=0.5236 effort=160 velocity=5.8
- joint RLEG_HIP_R: limit lower=0 upper=0 effort=30 velocity=0 -> lower=-0.349065850399 upper=1.57079632679 effort=100 velocity=3.87
- joint RLEG_HIP_Y: limit lower=0 upper=0 effort=30 velocity=0 -> lower=-2.095 upper=0.7 effort=160 velocity=5.8
- joint RLEG_KNEE: limit lower=0 upper=0 effort=30 velocity=0 -> lower=0 upper=2.618 effort=300 velocity=7

Commit message: Add visual information in URDF for visualization.

File: urdf/simple_humanoid.urdf (robot description, URDF)
Before this commit: robot simple_humanoid, 31 links, 30 joints
Links:
- link BODY: geometry visual box size=0.05 0.05 0.111; visual box size=0.08 0.08 0.08
- link LARM_LINK1: geometry visual cylinder length=0.05 radius=0.025
- link LARM_LINK2: geometry visual box size=0.05 0.05 0.163; visual cylinder length=0.05 radius=0.025
- link LARM_LINK3: geometry visual cylinder length=0.05 radius=0.025
- link LARM_LINK4: geometry visual box size=0.05 0.05 0.147; visual cylinder length=0.05 radius=0.025
- link LARM_LINK5: geometry visual cylinder length=0.05 radius=0.025
- link LARM_LINK6: geometry visual box size=0.05 0.03 0.175; visual cylinder length=0.05 radius=0.025
- link LLEG_LINK1: geometry visual cylinder length=0.1 radius=0.05
- link LLEG_LINK2: geometry visual cylinder length=0.1 radius=0.05
- link LLEG_LINK3: geometry visual box size=0.1 0.1 0.1535; visual cylinder length=0.1 radius=0.05
- link LLEG_LINK4: geometry visual box size=0.1 0.1 0.2; visual cylinder length=0.1 radius=0.05
- link LLEG_LINK5: geometry visual cylinder length=0.1 radius=0.05
- link RLEG_LINK1: geometry visual cylinder length=0.1 radius=0.05
- link RLEG_LINK2: geometry visual cylinder length=0.1 radius=0.05
- link RLEG_LINK3: geometry visual box size=0.1 0.1 0.1535; visual cylinder length=0.1 radius=0.05
- link RLEG_LINK4: geometry visual box size=0.1 0.1 0.2; visual cylinder length=0.1 radius=0.05
- link RLEG_LINK5: geometry visual cylinder length=0.1 radius=0.05
- link WAIST_LINK1: geometry visual cylinder length=0.05 radius=0.025
- link WAIST_LINK2: geometry visual box size=0.05 0.05 0.275; visual cylinder length=0.05 radius=0.025
- link l_ankle: geometry visual box size=0.25 0.14 0.02; visual cylinder length=0.1 radius=0.05
- link l_wrist: geometry visual box size=0.05 0.03 0.15
- link r_ankle: geometry visual box size=0.25 0.14 0.02; visual cylinder length=0.1 radius=0.05
- link torso: geometry visual box size=0.05 0.05 0.03; visual box size=0.15 0.27 0.05

Commit message: Add right arm visuals

File: urdf/simple_humanoid.urdf (robot description, URDF)
Before this commit: robot simple_humanoid, 31 links, 30 joints
Links:
- link RARM_LINK1: geometry visual cylinder length=0.05 radius=0.025
- link RARM_LINK2: geometry visual box size=0.05 0.05 0.163; visual cylinder length=0.05 radius=0.025
- link RARM_LINK3: geometry visual cylinder length=0.05 radius=0.025
- link RARM_LINK4: geometry visual box size=0.05 0.05 0.147; visual cylinder length=0.05 radius=0.025
- link RARM_LINK5: geometry visual cylinder length=0.05 radius=0.025
- link RARM_LINK6: geometry visual box size=0.05 0.03 0.175; visual cylinder length=0.05 radius=0.025
- link r_wrist: geometry visual box size=0.05 0.03 0.15
